Commit message: update pid

File: src/car_scale_description/urdf/camera.xacro (robot description, xacro)
@@ -3,19 +3,20 @@
 <link name = "camera_link_optical"/>
 <joint name = "camera_optical_joint" type="fixed">
-    <origin xyz = "0 0 0" rpy ="${-pi/2} 0 ${-pi/2}"/>
+    <!-- <origin xyz = "0.15 0 0" rpy ="0 ${+pi/6} 0"/> -->
+    <origin xyz = "0.15 0 0" rpy ="0 0 0"/>
     <parent link = "ras_camera_1"/>
     <child link="camera_link_optical"/>
 </joint>
-<gazebo reference ="ras_camera_1">
+<gazebo reference ="camera_link_optical">
     <sensor name="camera_sensor" type="camera">
         <camera>
-            <horizontal_fov>1.3962634</horizontal_fov>
+            <horizontal_fov>1.085</horizontal_fov> <!-- 62.2 degrees = 1.085 rad -->
             <image>
-                <width>640</width>
-                <height>480</height>
+                <width>3280</width>
+                <height>2464</height>
                 <format>R8G8B8</format>
             </image>
             <clip>
-                <near>0.1</near>
+                <near>0.01</near> <!-- closer, better for small scenes -->
                 <far>100</far>
             </clip>
@@ -23,5 +24,5 @@
                 <type>gaussian</type>
                 <mean>0.0</mean>
-                <stddev>0.01</stddev>
+                <stddev>0.005</stddev> <!-- Less noise, PiCam is quite clean -->
             </noise>
             <optical_frame_id>camera_link_optical</optical_frame_id>
@@ -29,5 +30,5 @@
         </camera>
         <always_on>1</always_on>
-        <update_rate>30</update_rate>
+        <update_rate>30</update_rate> <!-- 30 FPS -->
         <visualize>true</visualize>
         <topic>camera/image_raw</topic>

File: src/car_scale_description/urdf/car_scale.xacro (robot description, xacro)
@@ -1,9 +1,9 @@
 <?xml version="1.0" ?>
 <robot name="car_scale" xmlns:xacro="http://www.ros.org/wiki/xacro">
-  <xacro:include filename="$(find car_scale_description)/urdf/car_footprint.xacro" />
-  <xacro:include filename="$(find car_scale_description)/urdf/materials.xacro" />
-  <xacro:include filename="$(find car_scale_description)/urdf/car_scale.trans" />
-  <xacro:include filename="$(find car_scale_description)/urdf/car_scale.gazebo" />
-  <xacro:include filename="$(find car_scale_description)/urdf/camera.xacro" />
+<xacro:include filename="$(find car_scale_description)/urdf/camera.xacro" />
+<xacro:include filename="$(find car_scale_description)/urdf/car_footprint.xacro" />
+<xacro:include filename="$(find car_scale_description)/urdf/materials.xacro" />
+<xacro:include filename="$(find car_scale_description)/urdf/car_scale.trans" />
+<xacro:include filename="$(find car_scale_description)/urdf/car_scale.gazebo" />
 <link name="base_link">
   <inertial>
@@ -266,24 +266,4 @@
   </collision>
 </link>
-<link name="ras_camera_1">
-  <inertial>
-    <origin xyz="0.01391268653175004 0.10434306470190896 -0.10389239095408831" rpy="0 0 0"/>
-    <mass value="6.74286978494596"/>
-    <inertia ixx="0.049747" iyy="0.027218" izz="0.025635" ixy="2.5e-05" iyz="0.000336" ixz="0.000816"/>
-  </inertial>
-  <visual>
-    <origin xyz="-0.488158 0.479042 -1.51315" rpy="0 0 0"/>
-    <geometry>
-      <mesh filename="file://$(find car_scale_description)/meshes/ras_camera_1.stl" scale="0.001 0.001 0.001"/>
-    </geometry>
-    <material name="silver"/>
-  </visual>
-  <collision>
-    <origin xyz="-0.488158 0.479042 -1.51315" rpy="0 0 0"/>
-    <geometry>
-      <mesh filename="file://$(find car_scale_description)/meshes/ras_camera_1.stl" scale="0.001 0.001 0.001"/>
-    </geometry>
-  </collision>
-</link>
 <link name="raspberry_1">
   <inertial>
@@ -308,7 +288,7 @@
 <link name="base_camera_1">
   <inertial>
-    <origin xyz="-7.22659181939811e-08 -4.208437758279615e-07 0.45457683334028" rpy="0 0 0"/>
-    <mass value="48.35634401680473"/>
-    <inertia ixx="4.857732" iyy="4.389906" izz="0.649878" ixy="0.0" iyz="-0.0" ixz="-0.0"/>
+    <origin xyz="0.006164669793814914 -4.2085712453898694e-07 0.28276397732579905" rpy="0 0 0"/>
+    <mass value="31.13802766340137"/>
+    <inertia ixx="1.738526" iyy="1.384342" izz="0.475699" ixy="0.0" iyz="-0.0" ixz="-0.072073"/>
   </inertial>
   <visual>
@@ -323,4 +303,24 @@
     <geometry>
       <mesh filename="file://$(find car_scale_description)/meshes/base_camera_1.stl" scale="0.001 0.001 0.001"/>
+    </geometry>
+  </collision>
+</link>
+<link name="ras_camera_1">
+  <inertial>
+    <origin xyz="-0.04808730656914956 -0.0006569352980925203 0.021607609045916965" rpy="0 0 0"/>
+    <mass value="6.74286978494596"/>
+    <inertia ixx="0.049747" iyy="0.027218" izz="0.025635" ixy="2.5e-05" iyz="0.000336" ixz="0.000816"/>
+  </inertial>
+  <visual>
+    <origin xyz="-0.488158 0.374042 -1.18765" rpy="0 0 0"/>
+    <geometry>
+      <mesh filename="file://$(find car_scale_description)/meshes/ras_camera_1.stl" scale="0.001 0.001 0.001"/>
+    </geometry>
+    <material name="silver"/>
+  </visual>
+  <collision>
+    <origin xyz="-0.488158 0.374042 -1.18765" rpy="0 0 0"/>
+    <geometry>
+      <mesh filename="file://$(find car_scale_description)/meshes/ras_camera_1.stl" scale="0.001 0.001 0.001"/>
     </geometry>
   </collision>
@@ -390,9 +390,4 @@
   <child link="base_battery_1"/>
 </joint>
-<joint name="Rigid 39" type="fixed">
-  <origin xyz="0.075 -0.105 1.0" rpy="0 0 0"/>
-  <parent link="base_camera_1"/>
-  <child link="ras_camera_1"/>
-</joint>
 <joint name="Rigid 40" type="fixed">
   <origin xyz="0.3325 -0.245 0.86" rpy="0 0 0"/>
@@ -400,8 +395,13 @@
   <child link="raspberry_1"/>
 </joint>
-<joint name="Rigid 41" type="fixed">
+<joint name="Rigid 42" type="fixed">
   <origin xyz="0.413158 -0.374042 0.51315" rpy="0 0 0"/>
   <parent link="base_link"/>
   <child link="base_camera_1"/>
 </joint>
+<joint name="Rigid 45" type="fixed">
+  <origin xyz="0.075 0.0 0.6745" rpy="0 0 0"/>
+  <parent link="base_camera_1"/>
+  <child link="ras_camera_1"/>
+</joint>
 </robot>
